Commit message: Tune parameters

File: cartographer_ros/urdf/itri_van.urdf (robot description, URDF)
Before this commit: robot itri_van, 5 links, 4 joints
Joints:
- joint car_to_gps: origin xyz=-0.12 0.27 0.96 -> xyz=-0.12 0 -0.64
- joint car_to_imu_mount: origin xyz=0.15 0 -0.3 rpy=0 0 0 -> xyz=0.15 0 -1.9 rpy=0 0 0
- joint car_to_lidar: origin xyz=0 0 1.5 -> xyz=0 0 0 rpy=0 0 -2.15
